File: hardware/hardware.kicad_pcb (KiCad board)
At the start: 2 copper layers, 40 parts, among them J1 Screw_Terminal_1x03, J2 Screw_Terminal_1x03, P1 CONN_01X02, P2 CONN_01X08, Q0 BSS138, Q1 BSS138, Q2 BSS138, U1 WeMos_mini, U2 75LBC176

Commit message: Added systemd service
Parts:
- C1: value C -> 2.2u
- C2, C3, C4: value C -> 100n
- Q0, Q1, Q2: value BSS138 -> 2n7002
- R0, R1, R11, R2, R3, R4, R5: value R -> 2k2
- R10: value R -> 120R
- R6, R9: value R -> 150R
- R7, R8: value R -> 10R
Other:
- board outline added: 85.2 x 39.6 mm
Changed lines of the file:
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@@
     (links 69)
     (no_connects 10)
-    (area 127.057199 80.078866 212.852001 120.142001)
+    (area 127.584999 80.467999 212.927401 120.217401)
     (thickness 1.6)
-    (drawings 0)
+    (drawings 4)
     (tracks 183)
     (zones 0)
@@
     (last_trace_width 0.762)
     (trace_clearance 0.3048)
-    (zone_clearance 0.508)
+    (zone_clearance 0.3048)
     (zone_45_only yes)
     (trace_min 0.2)
@@
     (pad_drill 0.6)
     (pad_to_mask_clearance 0)
-    (aux_axis_origin 0 0)
+    (aux_axis_origin 203.327 87.249)
     (grid_origin 217.297 108.585)
     (visible_elements FFFFFFFF)
     (pcbplotparams
-      (layerselection 0x00030_80000001)
+      (layerselection 0x01000_80000001)
       (usegerberextensions false)
       (excludeedgelayer true)
@@
       (outputformat 1)
       (mirror false)
-      (drillshape 1)
+      (drillshape 0)
       (scaleselection 1)
-      (outputdirectory ""))
+      (outputdirectory fabric/))
   )
   (net 0 "")
@@
       (effects (font (size 1 1) (thickness 0.15)))
     )
-    (fp_text value R (at -0.39878 4.20116 180) (layer F.Fab)
+    (fp_text value 150R (at -0.39878 4.20116 180) (layer F.Fab)
       (effects (font (size 1 1) (thickness 0.15)))
     )
@@
       (effects (font (size 1 1) (thickness 0.15)))
     )
-    (fp_text value R (at -0.39878 4.20116 90) (layer F.Fab)
+    (fp_text value 120R (at -0.39878 4.20116 90) (layer F.Fab)
       (effects (font (size 1 1) (thickness 0.15)))
     )
@@
       (effects (font (size 1 1) (thickness 0.15)) (justify mirror))
     )
-    (fp_text value BSS138 (at 0 -2.5) (layer B.Fab)
+    (fp_text value 2n7002 (at 0 -2.5) (layer B.Fab)
       (effects (font (size 1 1) (thickness 0.15)) (justify mirror))
     )
@@
       (effects (font (size 1 1) (thickness 0.15)) (justify mirror))
     )
-    (fp_text value BSS138 (at 0 -2.5) (layer B.Fab)
+    (fp_text value 2n7002 (at 0 -2.5) (layer B.Fab)
       (effects (font (size 1 1) (thickness 0.15)) (justify mirror))
     )
@@
       (effects (font (size 1 1) (thickness 0.15)) (justify mirror))
     )
-    (fp_text value BSS138 (at 0 -2.5) (layer B.Fab)
+    (fp_text value 2n7002 (at 0 -2.5) (layer B.Fab)
       (effects (font (size 1 1) (thickness 0.15)) (justify mirror))
     )
@@
       (effects (font (size 1 1) (thickness 0.15)) (justify mirror))
     )
-    (fp_text value R (at 0 -2.1 90) (layer B.Fab)
+    (fp_text value 2k2 (at 0 -2.1 90) (layer B.Fab)
       (effects (font (size 1 1) (thickness 0.15)) (justify mirror))
     )
@@
       (effects (font (size 1 1) (thickness 0.15)) (justify mirror))
     )
-    (fp_text value R (at 0 -2.1 180) (layer B.Fab)
+    (fp_text value 2k2 (at 0 -2.1 180) (layer B.Fab)
       (effects (font (size 1 1) (thickness 0.15)) (justify mirror))
     )
@@
       (effects (font (size 1 1) (thickness 0.15)) (justify mirror))
     )
-    (fp_text value R (at 0 -2.1 90) (layer B.Fab)
+    (fp_text value 2k2 (at 0 -2.1 90) (layer B.Fab)
       (effects (font (size 1 1) (thickness 0.15)) (justify mirror))
     )
@@
       (effects (font (size 1 1) (thickness 0.15)) (justify mirror))
     )
-    (fp_text value R (at 0 -2.1 180) (layer B.Fab)
+    (fp_text value 2k2 (at 0 -2.1 180) (layer B.Fab)
       (effects (font (size 1 1) (thickness 0.15)) (justify mirror))
     )
@@
       (effects (font (size 1 1) (thickness 0.15)) (justify mirror))
     )
-    (fp_text value R (at 0 -2.1 180) (layer B.Fab)
+    (fp_text value 2k2 (at 0 -2.1 180) (layer B.Fab)
       (effects (font (size 1 1) (thickness 0.15)) (justify mirror))
     )
@@
       (effects (font (size 1 1) (thickness 0.15)) (justify mirror))
     )
-    (fp_text value C (at 0 -2.1 90) (layer B.Fab)
+    (fp_text value 2.2u (at 0 -2.1 90) (layer B.Fab)
       (effects (font (size 1 1) (thickness 0.15)) (justify mirror))
     )
@@
       (effects (font (size 1 1) (thickness 0.15)) (justify mirror))
     )
-    (fp_text value C (at 0 -2.1 90) (layer B.Fab)
+    (fp_text value 100n (at 0 -2.1 90) (layer B.Fab)
       (effects (font (size 1 1) (thickness 0.15)) (justify mirror))
     )
@@
       (effects (font (size 1 1) (thickness 0.15)) (justify mirror))
     )
-    (fp_text value C (at 0 -2.1 180) (layer B.Fab)
+    (fp_text value 100n (at 0 -2.1 180) (layer B.Fab)
       (effects (font (size 1 1) (thickness 0.15)) (justify mirror))
     )
@@
       (effects (font (size 1 1) (thickness 0.15)) (justify mirror))
     )
-    (fp_text value C (at 0 -2.3) (layer B.Fab)
+    (fp_text value 100n (at 0 -2.3) (layer B.Fab)
       (effects (font (size 1 1) (thickness 0.15)) (justify mirror))
     )
@@
       (effects (font (size 1 1) (thickness 0.15)))
     )
-    (fp_text value R (at -0.39878 4.20116 180) (layer F.Fab)
+    (fp_text value 150R (at -0.39878 4.20116 180) (layer F.Fab)
       (effects (font (size 1 1) (thickness 0.15)))
     )
@@
       (effects (font (size 1 1) (thickness 0.15)))
     )
-    (fp_text value R (at -0.39878 4.20116 180) (layer F.Fab)
+    (fp_text value 10R (at -0.39878 4.20116 180) (layer F.Fab)
       (effects (font (size 1 1) (thickness 0.15)))
     )
@@
       (effects (font (size 1 1) (thickness 0.15)))
     )
-    (fp_text value R (at -0.39878 4.20116 180) (layer F.Fab)
+    (fp_text value 10R (at -0.39878 4.20116 180) (layer F.Fab)
       (effects (font (size 1 1) (thickness 0.15)))
     )
@@
       (effects (font (size 1 1) (thickness 0.15)) (justify mirror))
     )
-    (fp_text value R (at 0 -2.1 270) (layer B.Fab)
+    (fp_text value 2k2 (at 0 -2.1 270) (layer B.Fab)
       (effects (font (size 1 1) (thickness 0.15)) (justify mirror))
     )
@@
       (effects (font (size 1 1) (thickness 0.15)) (justify mirror))
     )
-    (fp_text value R (at 0 -2.1 90) (layer B.Fab)
+    (fp_text value 2k2 (at 0 -2.1 90) (layer B.Fab)
       (effects (font (size 1 1) (thickness 0.15)) (justify mirror))
     )
@@
       (net 9 GND))
   )
+  (gr_line (start 212.8774 120.1674) (end 127.635 120.1674) (angle 90) (layer Edge.Cuts) (width 0.1))
+  (gr_line (start 127.635 80.518) (end 127.635 120.142) (layer Edge.Cuts) (width 0.1))
+  (gr_line (start 212.852 80.518) (end 127.635 80.518) (layer Edge.Cuts) (width 0.1))
+  (gr_line (start 212.852 120.142) (end 212.852 80.518) (layer Edge.Cuts) (width 0.1))
   (via (at 163.068 101.219) (size 0.6) (drill 0.4) (layers F.Cu B.Cu) (net 1))
   (segment (start 163.068 104.394) (end 163.068 101.219) (width 0.762) (layer F.Cu) (net 1))
@@
   (segment (start 136.3345 92.837) (end 136.398 92.7735) (width 0.762) (layer B.Cu) (net 24))
   (zone (net 9) (net_name GND) (layer B.Cu) (hatch edge 0.508)
-    (connect_pads (clearance 0.508))
+    (connect_pads (clearance 0.3048))
     (min_thickness 0.254)
-    (fill yes (arc_segments 16) (thermal_gap 0.508) (thermal_bridge_width 0.508))
+    (fill yes (arc_segments 32) (thermal_gap 0.508) (thermal_bridge_width 0.508))
     (polygon
       (pts
