File: hardware/v2/_autosave-hardware.kicad_pcb (KiCad board)
At the start: 2 copper layers, 87.8 x 43.5 mm, 43 parts, among them J1 Screw_Terminal_1x03, J2 Screw_Terminal_01x02, J3 Screw_Terminal_1x03, J4 Barrel_Jack_Switch, J5 Screw_Terminal_01x02, J6 Screw_Terminal_01x02, J7 Screw_Terminal_01x02, P1 CONN_01X02, P2 CONN_01X08, Q0 2n7002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

Commit message: PCB V2
Parts:
- moved J4 6.70 mm to (208.5, 110.1)
- moved R7 0.33 mm to (193.7, 87.0)
Routing:
- net Net-(D3-Pad2): track 5.35 -> 17.0 mm
- net GND: track 207.7 -> 217.6 mm
Other:
- board size 87.8 x 43.5 mm -> 109.6 x 44.2 mm
Changed lines of the file:
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@@
     (thickness 1.6)
     (drawings 5)
-    (tracks 267)
+    (tracks 265)
     (zones 0)
     (modules 43)
@@
     (aux_axis_origin 203.327 87.249)
     (grid_origin 217.297 108.585)
-    (visible_elements 7FFFFFFF)
+    (visible_elements 7FFFEFFF)
     (pcbplotparams
       (layerselection 0x01000_80000001)
@@
   )
   (module Connector_BarrelJack:BarrelJack_Horizontal (layer F.Cu)
-    (at 207.5942 103.4796 90)
+    (at 208.534 110.109 90)
     (descr "DC Barrel Jack")
     (tags "Power Jack")
@@
   )
   (module Resistor_THT:R_Axial_DIN0207_L6.3mm_D2.5mm_P10.16mm_Horizontal (layer F.Cu)
-    (at 193.675 86.6648 270)
+    (at 193.675 86.995 270)
     (descr "Resistor, Axial_DIN0207 series, Axial, Horizontal, pin pitch=10.16mm, 0.25W = 1/4W, length*diameter=6.3*2.5mm^2, http://cdn-reichelt.de/documents/datenblatt/B400/1_4W%23YAG.pdf")
     (tags "Resistor Axial_DIN0207 series Axial Horizontal pin pitch 10.16mm 0.25W = 1/4W length 6.3mm diameter 2.5mm")
@@
     )
   )
-  (gr_line (start 215.2142 124.1298) (end 127.6096 124.0282) (layer Edge.Cuts) (width 0.1))
+  (gr_line (start 215.265 124.714) (end 105.7148 124.9172) (layer Edge.Cuts) (width 0.1))
   (gr_poly (pts (xy 202.379026 117.912789) (xy 202.379026 101.148789) (xy 180.281026 101.148789) (xy 180.281026 117.912789)) (layer Margin) (width 0.15))
-  (gr_line (start 127.508 80.899) (end 127.6604 123.9266) (layer Edge.Cuts) (width 0.1))
+  (gr_line (start 127.254 80.899) (end 127.127 124.587) (layer Edge.Cuts) (width 0.1))
   (gr_line (start 215.138 80.6704) (end 127.508 80.8482) (layer Edge.Cuts) (width 0.1))
-  (gr_line (start 215.2904 124.1298) (end 215.138 80.6704) (layer Edge.Cuts) (width 0.1))
+  (gr_line (start 215.265 124.841) (end 215.138 80.6704) (layer Edge.Cuts) (width 0.1))
   (via (at 161.9504 101.219) (size 0.6) (drill 0.4) (layers F.Cu B.Cu) (net 1))
   (segment (start 161.9504 104.394) (end 161.9504 101.219) (width 0.762) (layer F.Cu) (net 1))
@@
   (segment (start 176.3624 93.98) (end 176.3624 98.425) (width 0.762) (layer B.Cu) (net 4))
   (segment (start 179.2224 93.98) (end 179.30114 93.98) (width 0.762) (layer B.Cu) (net 4))
-  (segment (start 179.2986 93.9038) (end 179.2224 93.98) (width 0.762) (layer B.Cu) (net 4))
-  (segment (start 179.2986 91.2712) (end 179.2986 93.9038) (width 0.762) (layer B.Cu) (net 4))
-  (segment (start 180.7882 91.2712) (end 179.2986 91.2712) (width 0.762) (layer B.Cu) (net 4))
-  (segment (start 182.45983 83.058) (end 181.3306 84.18723) (width 0.762) (layer B.Cu) (net 4))
-  (segment (start 183.5912 83.058) (end 182.45983 83.058) (width 0.762) (layer B.Cu) (net 4))
-  (segment (start 181.3306 90.7288) (end 180.7882 91.2712) (width 0.762) (layer B.Cu) (net 4))
-  (segment (start 181.3306 84.18723) (end 181.3306 90.7288) (width 0.762) (layer B.Cu) (net 4))
   (segment (start 154.2542 119.507) (end 150.7744 119.507) (width 0.762) (layer B.Cu) (net 4))
   (segment (start 176.8999 107.3859) (end 176.6914 107.5944) (width 0.762) (layer B.Cu) (net 4))
@@
   (segment (start 158.1404 110.5535) (end 159.0421 109.6518) (width 0.762) (layer B.Cu) (net 4))
   (segment (start 159.0421 109.6518) (end 162.1282 109.6518) (width 0.762) (layer B.Cu) (net 4))
+  (segment (start 182.45983 83.058) (end 183.5912 83.058) (width 0.762) (layer B.Cu) (net 4))
+  (segment (start 181.3306 84.18723) (end 182.45983 83.058) (width 0.762) (layer B.Cu) (net 4))
+  (segment (start 181.3306 93.00317) (end 181.3306 84.18723) (width 0.762) (layer B.Cu) (net 4))
+  (segment (start 180.35377 93.98) (end 181.3306 93.00317) (width 0.762) (layer B.Cu) (net 4))
+  (segment (start 179.2224 93.98) (end 180.35377 93.98) (width 0.762) (layer B.Cu) (net 4))
   (segment (start 158.1404 92.7735) (end 160.3629 92.7735) (width 0.762) (layer B.Cu) (net 5))
   (segment (start 161.2544 102.555) (end 163.9824 102.555) (width 0.762) (layer B.Cu) (net 5))
@@
   (segment (start 137.6934 91.44) (end 136.5504 90.297) (width 0.762) (layer B.Cu) (net 9))
   (segment (start 138.2014 91.948) (end 137.6934 91.44) (width 0.762) (layer B.Cu) (net 9))
-  (segment (start 177.6386 89.2212) (end 176.5554 88.138) (width 0.762) (layer B.Cu) (net 9))
-  (segment (start 179.2986 89.2212) (end 177.6386 89.2212) (width 0.762) (layer B.Cu) (net 9))
   (segment (start 136.0678 113.266) (end 136.8626 112.4712) (width 0.762) (layer B.Cu) (net 9))
   (segment (start 136.0678 114.6048) (end 136.0678 113.266) (width 0.762) (layer B.Cu) (net 9))
@@
   (segment (start 200.7108 110.5752) (end 200.7108 113.538) (width 0.762) (layer B.Cu) (net 9))
   (segment (start 200.7362 113.5634) (end 200.7362 116.1034) (width 0.762) (layer B.Cu) (net 9))
-  (segment (start 203.5104 113.5634) (end 207.5942 109.4796) (width 0.762) (layer B.Cu) (net 9))
-  (segment (start 200.7362 113.5634) (end 203.5104 113.5634) (width 0.762) (layer B.Cu) (net 9))
-  (segment (start 210.5942 106.4796) (end 207.5942 109.4796) (width 0.762) (layer B.Cu) (net 9))
-  (segment (start 212.2942 106.4796) (end 210.5942 106.4796) (width 0.762) (layer B.Cu) (net 9))
   (segment (start 171.5589 108.0135) (end 173.3042 106.2682) (width 0.762) (layer B.Cu) (net 9))
   (segment (start 158.1404 108.0135) (end 171.5589 108.0135) (width 0.762) (layer B.Cu) (net 9))
@@
   (segment (start 134.9756 113.5126) (end 136.0678 114.6048) (width 0.762) (layer B.Cu) (net 9))
   (segment (start 133.867 113.5126) (end 134.9756 113.5126) (width 0.762) (layer B.Cu) (net 9))
+  (segment (start 131.5212 90.297) (end 128.016 93.8022) (width 0.762) (layer B.Cu) (net 9))
+  (segment (start 128.016 93.8022) (end 128.016 116.459) (width 0.762) (layer B.Cu) (net 9))
   (segment (start 168.7924 99.06) (end 171.6024 99.06) (width 0.762) (layer B.Cu) (net 10))
   (segment (start 171.6024 96.52) (end 171.6024 99.06) (width 0.762) (layer B.Cu) (net 10))
@@
   (segment (start 135.2931 95.3008) (end 135.2804 95.3135) (width 0.762) (layer B.Cu) (net 24))
   (segment (start 138.7762 95.3008) (end 135.2931 95.3008) (width 0.762) (layer B.Cu) (net 24))
-  (segment (start 131.5212 95.377) (end 129.4892 95.377) (width 0.762) (layer B.Cu) (net 24))
-  (segment (start 128.8034 96.0628) (end 129.4892 95.377) (width 0.762) (layer B.Cu) (net 24))
-  (segment (start 128.8542 113.5126) (end 128.8034 113.4618) (width 0.762) (layer B.Cu) (net 24))
-  (segment (start 131.817 113.5126) (end 128.8542 113.5126) (width 0.762) (layer B.Cu) (net 24))
-  (segment (start 128.8034 113.4618) (end 128.8034 96.0628) (width 0.762) (layer B.Cu) (net 24))
-  (segment (start 128.8034 113.6904) (end 134.62 119.507) (width 0.762) (layer B.Cu) (net 24))
-  (segment (start 128.8034 113.4618) (end 128.8034 113.6904) (width 0.762) (layer B.Cu) (net 24))
+  (segment (start 134.62 118.491) (end 134.62 119.507) (width 0.762) (layer B.Cu) (net 24))
+  (segment (start 129.286 113.157) (end 131.064 114.935) (width 0.762) (layer B.Cu) (net 24))
+  (segment (start 129.286 96.410119) (end 129.286 113.157) (width 0.762) (layer B.Cu) (net 24))
+  (segment (start 130.319119 95.377) (end 129.286 96.410119) (width 0.762) (layer B.Cu) (net 24))
+  (segment (start 131.5212 95.377) (end 130.319119 95.377) (width 0.762) (layer B.Cu) (net 24))
+  (segment (start 131.064 114.935) (end 134.62 118.491) (width 0.762) (layer B.Cu) (net 24))
+  (segment (start 129.6416 113.5126) (end 131.064 114.935) (width 0.762) (layer B.Cu) (net 24))
+  (segment (start 131.817 113.5126) (end 129.6416 113.5126) (width 0.762) (layer B.Cu) (net 24))
   (segment (start 138.1432 114.6302) (end 138.1178 114.6048) (width 0.762) (layer B.Cu) (net 26))
   (segment (start 138.1432 116.9416) (end 138.1432 114.6302) (width 0.762) (layer B.Cu) (net 26))
@@
   (segment (start 200.7452 102.782615) (end 200.601026 102.926789) (width 0.762) (layer B.Cu) (net 31))
   (segment (start 200.7452 99.187) (end 200.7452 102.782615) (width 0.762) (layer B.Cu) (net 31))
-  (segment (start 205.0452 100.9306) (end 207.5942 103.4796) (width 0.762) (layer B.Cu) (net 32))
   (segment (start 205.0452 99.187) (end 205.0452 100.9306) (width 0.762) (layer B.Cu) (net 32))
+  (segment (start 208.534 107.597) (end 206.474 105.537) (width 0.762) (layer B.Cu) (net 32))
+  (segment (start 208.534 110.109) (end 208.534 107.597) (width 0.762) (layer B.Cu) (net 32))
+  (segment (start 205.0452 104.1082) (end 208.534 107.597) (width 0.762) (layer B.Cu) (net 32))
+  (segment (start 205.0452 99.187) (end 205.0452 104.1082) (width 0.762) (layer B.Cu) (net 32))
   (segment (start 136.67 119.507) (end 141.8844 119.507) (width 0.762) (layer B.Cu) (net 34))
   (segment (start 136.67 118.7376) (end 136.67 119.507) (width 0.762) (layer B.Cu) (net 34))
@@
     (polygon
       (pts
-        (xy 127.257889 80.794225) (xy 216.578023 80.75295) (xy 216.6366 124.2314) (xy 127.402511 123.955175) (xy 126.8476 104.5464)
+        (xy 126.111 80.772) (xy 216.578023 80.75295) (xy 216.535 124.587) (xy 126.492 124.714) (xy 126.492 122.936)
       )
     )
