File: hardware/v2/hardware.kicad_pcb (KiCad board)
At the start: 2 copper layers, 89.2 x 43 mm, 43 parts, among them J1 Screw_Terminal_1x03, J2 Screw_Terminal_01x02, J3 Screw_Terminal_1x03, J4 Barrel_Jack_Switch, J5 Screw_Terminal_01x02, J6 Screw_Terminal_01x02, J7 Screw_Terminal_01x02, P1 CONN_01X02, P2 CONN_01X08, Q0 2n7002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

Commit message: Board texts
Parts:
- added H1: MountingHole, MountingHole:MountingHole_2.2mm_M2, F.Cu at (130.2, 82.7)
- added H2: MountingHole, MountingHole:MountingHole_2.2mm_M2, F.Cu at (130.2, 120.3)
- added H3: MountingHole, MountingHole:MountingHole_2.2mm_M2, F.Cu at (214.0, 99.9)
Other:
- board text added: "A"
- board text added: "ANT"
- board text added: "B"
- board text added: "DG"
- board text added: "GND"
- board text added: "NC"
- board text added: "SO"
- board text added: "USB"
- board text added: "VCC"
Changed lines of the file:
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@@
   (general
     (thickness 1.6)
-    (drawings 5)
+    (drawings 15)
     (tracks 279)
     (zones 0)
-    (modules 43)
+    (modules 46)
     (nets 35)
   )
@@
   (module wemos_d1_mini:D1_mini_board (layer B.Cu)
     (at 146.7104 102.9335 180)
-    (fp_text reference U1 (at 0.5334 5.7785 180) (layer B.SilkS)
+    (fp_text reference U1 (at 0.5334 5.7785 180) (layer B.SilkS) hide
       (effects (font (size 1 1) (thickness 0.15)) (justify mirror))
     )
@@
       (effects (font (size 1 1) (thickness 0.15)) (justify mirror))
     )
-    (fp_text user WeMos (at 0 15.24 180) (layer B.SilkS)
+    (fp_text user WeMos (at 0 15.24 180) (layer B.SilkS) hide
       (effects (font (size 3 3) (thickness 0.15)) (justify mirror))
     )
@@
     (descr "simple 3-pin terminal block, pitch 5.08mm, revamped version of bornier3")
     (tags "terminal block bornier3")
-    (fp_text reference J3 (at 5.05 -4.65 180) (layer F.SilkS)
+    (fp_text reference J3 (at -3.4798 0.0762 180) (layer F.SilkS)
       (effects (font (size 1 1) (thickness 0.15)))
     )
@@
     (descr "Through hole straight pin header, 1x02, 2.54mm pitch, single row")
     (tags "Through hole pin header THT 1x02 2.54mm single row")
-    (fp_text reference P1 (at 0 -2.33 90) (layer F.SilkS)
+    (fp_text reference P1 (at -3.048 -0.1524 90) (layer F.SilkS)
       (effects (font (size 1 1) (thickness 0.15)))
     )
@@
     )
   )
+  (module MountingHole:MountingHole_2.2mm_M2 (layer F.Cu)
+    (at 130.175 82.677)
+    (descr "Mounting Hole 2.2mm, no annular, M2")
+    (tags "mounting hole 2.2mm no annular m2")
+    (attr virtual)
+    (fp_text reference H1 (at 3.302 -1.524) (layer F.SilkS) hide
+      (effects (font (size 1 1) (thickness 0.15)))
+    )
+    (fp_text value MountingHole (at 0 3.2) (layer F.Fab)
+      (effects (font (size 1 1) (thickness 0.15)))
+    )
+    (fp_circle (center 0 0) (end 2.45 0) (layer F.CrtYd) (width 0.05))
+    (fp_circle (center 0 0) (end 2.2 0) (layer Cmts.User) (width 0.15))
+    (fp_text user %R (at 0.3 0) (layer F.Fab)
+      (effects (font (size 1 1) (thickness 0.15)))
+    )
+    (pad 1 np_thru_hole circle (at 0 0) (size 2.2 2.2) (drill 2.2) (layers *.Cu *.Mask))
+  )
+  (module MountingHole:MountingHole_2.2mm_M2 (layer F.Cu)
+    (at 130.175 120.269)
+    (descr "Mounting Hole 2.2mm, no annular, M2")
+    (tags "mounting hole 2.2mm no annular m2")
+    (attr virtual)
+    (fp_text reference H2 (at 0 -3.2) (layer F.SilkS) hide
+      (effects (font (size 1 1) (thickness 0.15)))
+    )
+    (fp_text value MountingHole (at 0 3.2) (layer F.Fab)
+      (effects (font (size 1 1) (thickness 0.15)))
+    )
+    (fp_text user %R (at 0.3 0) (layer F.Fab)
+      (effects (font (size 1 1) (thickness 0.15)))
+    )
+    (fp_circle (center 0 0) (end 2.2 0) (layer Cmts.User) (width 0.15))
+    (fp_circle (center 0 0) (end 2.45 0) (layer F.CrtYd) (width 0.05))
+    (pad 1 np_thru_hole circle (at 0 0) (size 2.2 2.2) (drill 2.2) (layers *.Cu *.Mask))
+  )
+  (module MountingHole:MountingHole_2.2mm_M2 (layer F.Cu)
+    (at 213.995 99.949)
+    (descr "Mounting Hole 2.2mm, no annular, M2")
+    (tags "mounting hole 2.2mm no annular m2")
+    (attr virtual)
+    (fp_text reference H3 (at 0 -3.2) (layer F.SilkS) hide
+      (effects (font (size 1 1) (thickness 0.15)))
+    )
+    (fp_text value MountingHole (at 0 3.2) (layer F.Fab)
+      (effects (font (size 1 1) (thickness 0.15)))
+    )
+    (fp_text user %R (at 0.3 0) (layer F.Fab)
+      (effects (font (size 1 1) (thickness 0.15)))
+    )
+    (fp_circle (center 0 0) (end 2.2 0) (layer Cmts.User) (width 0.15))
+    (fp_circle (center 0 0) (end 2.45 0) (layer F.CrtYd) (width 0.05))
+    (pad 1 np_thru_hole circle (at 0 0) (size 2.2 2.2) (drill 2.2) (layers *.Cu *.Mask))
+  )
+  (gr_text GND (at 180.467 85.471) (layer F.SilkS)
+    (effects (font (size 1.5 1.5) (thickness 0.3)))
+  )
+  (gr_text DG (at 170.307 85.471) (layer F.SilkS)
+    (effects (font (size 1.5 1.5) (thickness 0.3)))
+  )
+  (gr_text ANT (at 135.001 85.979) (layer F.SilkS)
+    (effects (font (size 1.5 1.5) (thickness 0.3)))
+  )
+  (gr_text USB (at 144.907 112.649) (layer F.SilkS)
+    (effects (font (size 1.5 1.5) (thickness 0.3)))
+  )
+  (gr_text SO (at 162.941 110.363) (layer F.SilkS)
+    (effects (font (size 1.5 1.5) (thickness 0.3)))
+  )
+  (gr_text NC (at 168.275 110.363) (layer F.SilkS)
+    (effects (font (size 1.5 1.5) (thickness 0.3)))
+  )
+  (gr_text VCC (at 173.609 110.363) (layer F.SilkS)
+    (effects (font (size 1.5 1.5) (thickness 0.3)))
+  )
+  (gr_text B (at 212.979 94.361 90) (layer F.SilkS)
+    (effects (font (size 1.5 1.5) (thickness 0.3)))
+  )
+  (gr_text GND (at 212.979 88.773 90) (layer F.SilkS)
+    (effects (font (size 1.5 1.5) (thickness 0.3)))
+  )
+  (gr_text A (at 212.725 83.439 90) (layer F.SilkS)
+    (effects (font (size 1.5 1.5) (thickness 0.3)))
+  )
   (gr_line (start 127.5715 122.936) (end 216.662 122.9995) (layer Edge.Cuts) (width 0.1))
